Commit message: Add realtime IK solvers for arm-only and interpolation with parameterized configurations

File: ffw_description/urdf/common/follower/ffw_follower_body.xacro (robot description, xacro)
@@ -435,5 +435,5 @@
          <origin xyz="0.041004 0 -0.135" rpy="0 0 0" />
          <axis xyz="0 1 0" />
-         <limit velocity="4.8" effort="1000" lower="-2.9361" upper="1.0786" />
+         <limit velocity="4.8" effort="1000" lower="-2.9361" upper="0.1" />
          <dynamics damping="0.1" />
       </joint>
